File: Shémas/Shémas.kicad_pcb (KiCad board)
At the start: 2 copper layers, 0 parts

Commit message: Add files via upload
Parts:
- added C1: 10nF, Capacitor_SMD:C_0805_2012Metric_Pad1.18x1.45mm_HandSolder, B.Cu at (139.5, 70.6)
- added C10: 0.1uF, Capacitor_SMD:C_0805_2012Metric_Pad1.18x1.45mm_HandSolder, F.Cu at (113.9, 77.7)
- added C11: 0.1uF, Capacitor_SMD:C_0805_2012Metric_Pad1.18x1.45mm_HandSolder, B.Cu at (132.6, 70.0)
- added C12: 47pF, Capacitor_SMD:C_0805_2012Metric_Pad1.18x1.45mm_HandSolder, F.Cu at (101.8, 72.9)
- added C13: 47pF, Capacitor_SMD:C_0805_2012Metric_Pad1.18x1.45mm_HandSolder, F.Cu at (103.3, 64.5)
- added C14: EEE-FN1H680XP 68uF, Capacitor_SMD:CP_Elec_8x6.9, F.Cu at (130.7, 81.2)
- added C15: 10uF, Capacitor_SMD:C_0805_2012Metric_Pad1.18x1.45mm_HandSolder, B.Cu at (105.5, 86.2)
- added C16: EEEFH1H101L 100uF, KiCad:EEETC1V470P, F.Cu at (144.4, 68.7)
- added C3: 0.1uF, Capacitor_SMD:C_0805_2012Metric_Pad1.18x1.45mm_HandSolder, F.Cu at (127.8, 66.3)
- added C4: 1uF, Capacitor_SMD:C_0805_2012Metric_Pad1.18x1.45mm_HandSolder, F.Cu at (131.3, 72.0)
- added C5: 10uF, Capacitor_SMD:C_0805_2012Metric_Pad1.18x1.45mm_HandSolder, B.Cu at (101.0, 78.0)
- added C6: 10uF, Capacitor_SMD:C_0805_2012Metric_Pad1.18x1.45mm_HandSolder, B.Cu at (105.5, 82.6)
- added C7: 0.1uF, Capacitor_SMD:C_0805_2012Metric_Pad1.18x1.45mm_HandSolder, B.Cu at (100.9, 82.5)
- added C8: 0.1uF, Capacitor_SMD:C_0805_2012Metric_Pad1.18x1.45mm_HandSolder, F.Cu at (120.3, 77.5)
- added C9: 0.1uF, Capacitor_SMD:C_0805_2012Metric_Pad1.18x1.45mm_HandSolder, B.Cu at (104.3, 72.3)
- added D1: SS14FL, Diode_SMD:D_SOD-123F, F.Cu at (137.8, 73.2)
- added FB1: BLM18KG121TZ1D, Capacitor_SMD:C_0402_1005Metric, B.Cu at (102.3, 85.2)
- added G***: LOGO, lib kicad:imagesilk1, F.Cu at (118.3, 93.9)
- added G***: LOGO, LOGO, B.Cu at (145.0, 82.7)
- added G***: LOGO, LOGO, B.Cu at (154.4, 67.1)
- added G***: LOGO, LOGO, B.Cu at (135.5, 80.8)
- added G***: LOGO, LOGO, B.Cu at (144.4, 63.9)
- added J1: Conn_01x04_Socket, Connector_PinSocket_2.54mm:PinSocket_1x04_P2.54mm_Vertical, F.Cu at (98.5, 65.0)
- added J3: Conn_01x04_Socket, Connector_PinSocket_2.54mm:PinSocket_1x04_P2.54mm_Vertical, F.Cu at (151.6, 71.4)
- added J4: Conn_01x03_Socket, Connector_PinSocket_2.54mm:PinSocket_1x03_P2.54mm_Vertical, F.Cu at (97.3, 77.4)
- added L1: NPI31W470MTRF 47uH, Inductor_SMD:L_Bourns-SRR1005, F.Cu at (142.6, 81.0)
- added R1: 91Ω, Capacitor_SMD:C_0805_2012Metric_Pad1.18x1.45mm_HandSolder, F.Cu at (127.7, 63.5)
- added R10: 10Ω, Capacitor_SMD:C_0805_2012Metric_Pad1.18x1.45mm_HandSolder, F.Cu at (102.8, 67.7)
- added R11: 10Ω, Capacitor_SMD:C_0805_2012Metric_Pad1.18x1.45mm_HandSolder, F.Cu at (102.8, 69.8)
- added R12: 120Ω, Capacitor_SMD:C_0805_2012Metric_Pad1.18x1.45mm_HandSolder, F.Cu at (107.2, 68.4)
- added R2: 150Ω, Capacitor_SMD:C_0805_2012Metric_Pad1.18x1.45mm_HandSolder, F.Cu at (127.9, 69.8)
- added R3: 330Ω, Capacitor_SMD:C_0805_2012Metric_Pad1.18x1.45mm_HandSolder, B.Cu at (101.0, 75.8)
- added R4: 4.7k, Capacitor_SMD:C_0805_2012Metric_Pad1.18x1.45mm_HandSolder, B.Cu at (108.3, 78.4)
- added R5: 4.7k, Capacitor_SMD:C_0805_2012Metric_Pad1.18x1.45mm_HandSolder, B.Cu at (109.2, 84.6)
- added R6: 4.7k, Capacitor_SMD:C_0805_2012Metric_Pad1.18x1.45mm_HandSolder, B.Cu at (109.0, 63.0)
- added R7: 10k, Capacitor_SMD:C_0805_2012Metric_Pad1.18x1.45mm_HandSolder, B.Cu at (108.4, 74.1)
- added R8: 4.7k, Capacitor_SMD:C_0805_2012Metric_Pad1.18x1.45mm_HandSolder, F.Cu at (122.6, 84.2)
- added R9: 4.7k, Capacitor_SMD:C_0805_2012Metric_Pad1.18x1.45mm_HandSolder, F.Cu at (122.7, 80.8)
- added U1: MCP3221, Package_TO_SOT_SMD:TSOT-23-5, B.Cu at (105.1, 78.6)
- added U2: TCA9517, Package_SO:SOIC-8_3.9x4.9mm_P1.27mm, F.Cu at (116.6, 82.5)
- added U3: XIAO ESP32C3, Library:xiao esp32-c3, B.Cu at (120.7, 90.3)
- added U5: LM117_TO3, Package_TO_SOT_SMD:SOT-223-3_TabPin2, F.Cu at (134.4, 67.2)
- added U6: TJA1051T, Package_SO:SOIC-8_3.9x4.9mm_P1.27mm, B.Cu at (107.2, 68.3)
- added U7: LM2674M-5.0, Package_SO:SOIC-8_3.9x4.9mm_P1.27mm, B.Cu at (144.7, 72.8)
Routing:
- net GND: track 0.00 -> 85.9 mm, vias 0 -> 28
- net +5V: track 0.00 -> 72.9 mm, vias 0 -> 20
- net /TXD: track 0.00 -> 40.7 mm
- net +3.3V: track 0.00 -> 28.4 mm, vias 0 -> 9
- net /SCLB: track 0.00 -> 23.8 mm, vias 0 -> 1
- net /SDAA: track 0.00 -> 22.4 mm, vias 0 -> 1
- net Net-(D1-K): track 0.00 -> 21.7 mm, vias 0 -> 1
- net /SDAB: track 0.00 -> 20.7 mm, vias 0 -> 1
- net /EN: track 0.00 -> 11.7 mm
- net Net-(U5-ADJ): track 0.00 -> 10.9 mm
- net Net-(U6-CANL): track 0.00 -> 10.8 mm, vias 0 -> 1
- net /SCLA: track 0.00 -> 10.5 mm, vias 0 -> 1
- net Net-(U6-CANH): track 0.00 -> 9.54 mm, vias 0 -> 1
- net Net-(U1-AIN): track 0.00 -> 9.17 mm
- net Net-(J4-Pin_2): track 0.00 -> 7.55 mm
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- added copper zone on F.Cu, net +12V
- added copper zone on In2.Cu, net +3.3V
- added copper zone on In2.Cu, net +5V
- added copper zone on B.Cu, net +5VA
- added copper zone on B.Cu, net GND
- added copper zone on In1.Cu, net GND
- added copper zone on In2.Cu, net Net-(J1-Pin_2)
- added copper zone on In2.Cu, net Net-(J1-Pin_3)
Other:
- board outline added: 65 x 26 mm
- copper layers 2 -> 4
- board text added: "+5V"
- board text added: "12V"
- board text added: "AN"
- board text added: "CH"
- board text added: "CL"
- board text added: "GND"
- board text added: "Mamoune B. Carl-D A."
- board text added: "Module CAN"
- board text added: "PCB module CAN"
