File: Shémas/Shémas.kicad_sch (KiCad schematic)
At the start: 36 parts, among them U1 MCP3221, U2 TCA9517, U3 XIAO ESP32C3, U5 LM117_TO3, U6 TJA1051T, U7 LM2674M-5.0

Commit message: Add files via upload
Parts:
- removed C14, C2: 100uF, symbol Device:C
- added C14: EEE-FN1H680XP 68uF, Capacitor_SMD:CP_Elec_8x6.9, symbol EEEFH1H101L:EEEFH1H101L
- added C16: EEEFH1H101L 100uF, KiCad:EEETC1V470P, symbol EEEFH1H101L:EEEFH1H101L
- added J1, J3: Conn_01x04_Socket, Connector_PinSocket_2.54mm:PinSocket_1x04_P2.54mm_Vertical, symbol Connector:Conn_01x04_Socket
- added J4: Conn_01x03_Socket, Connector_PinSocket_2.54mm:PinSocket_1x03_P2.54mm_Vertical, symbol Connector:Conn_01x03_Socket
- C1, C10, C11, C15, C3, C4, C5, C6, C7, C8, C9, R1, R10, R11, R12, R2, R3, R4, R5, R6, R7, R8, R9: footprint (none) -> Capacitor_SMD:C_0805_2012Metric_Pad1.18x1.45mm_HandSolder
- C12, C13: value 30pF -> 47pF; footprint (none) -> Capacitor_SMD:C_0805_2012Metric_Pad1.18x1.45mm_HandSolder
- D1: value 1N5824 -> SS14FL; footprint Diode_THT:D_DO-201AD_P15.24mm_Horizontal -> Diode_SMD:D_SOD-123F
- FB1: footprint (none) -> Capacitor_SMD:C_0402_1005Metric
- L1: value 100 uH -> NPI31W470MTRF 47uH; footprint (none) -> Inductor_SMD:L_Bourns-SRR1005
- U3: footprint (none) -> Library:xiao esp32-c3
Connections:
- net +12V: now also C16.1, J1.1 (Pin_1), J3.1 (Pin_1)
- net +5V: now also C14.1, J4.1 (Pin_1)
- net GND: now also C14.2, C16.2, J1.4 (Pin_4), J3.4 (Pin_4), J4.3 (Pin_3)
- net RXD: now also U3.14 (D7_RX_GPIO20); no longer R6.1
- net TXD: now also R6.1; no longer U3.14 (D7_RX_GPIO20)
- net AN out: no longer names the net of R3.1
- net AN out: now also J4.2 (Pin_2)
- net CAN H: no longer names the net of C13.2, R10.2
- net CAN H: now also J1.2 (Pin_2), J3.2 (Pin_2)
- net CAN L: no longer names the net of C12.2, R11.2
- net CAN L: now also J1.3 (Pin_3), J3.3 (Pin_3)
Other:
- note added: "Alimentation"
- note added: "CAN transmitter"
- note added: "Changer le rx et le tx pour un gpio random https://www.google.com/search?sca_esv=b6ab 7d9e5410acba&q=esp32+tja1051+schematic&tbm =isch&source=lnms&sa=X&ved=2ahUKEwi4x6Kqpsm EAxVUE1kFHTseAYkQ0pQJegQICxAB&biw=1536&bih= 711&dpr=1.25#imgrc=Fj9Knx-6niDcOM"
- note added: "ESP32-C3 xiao"
- note added: "Entrée analogique et conversion numérique"
- note added: "Level shifter"
- note added: "Power"
- note added: "Réseau CAN"
- note removed: "condensateur 100uH electrolytic capacitor"
- note removed: "gauge fil pour connecteur connexion serpent"
- title: Formule SAE module CAN -> Formule SAE module CAN SCH
- moved on the sheet: C10, C11, C12, C13, C15, C5, C6, C7, C8, C9, FB1, R1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
