File: Matériel/PCB/Shémas.kicad_sch (KiCad schematic)
At the start: 39 parts, among them J1 Conn_01x04_Socket, J3 Conn_01x04_Socket, J4 Conn_01x03_Socket, U1 MCP3221, U2 TCA9517, U3 XIAO ESP32C3, U5 LM117_TO3, U6 TJA1051T, U7 LM2674M-5.0

Commit message: Add files via upload
Parts:
- FB1: footprint Capacitor_SMD:C_0402_1005Metric -> Capacitor_SMD:C_0603_1608Metric
Other:
- moved on the sheet: R1
Changed lines of the file:
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@@
     (stroke (width 0) (type default))
   )
-  (wire (pts (xy 140.462 171.069) (xy 140.462 172.085))
+  (wire (pts (xy 140.462 171.069) (xy 140.462 171.323))
     (stroke (width 0) (type default))
   )
@@
   )
   (wire (pts (xy 151.638 171.069) (xy 151.638 168.402))
-    (stroke (width 0) (type default))
-  )
-  (wire (pts (xy 140.462 179.705) (xy 140.462 178.943))
     (stroke (width 0) (type default))
   )
@@
     )
   )
-  (symbol (lib_id "Device:R") (at 140.462 175.895 0) (unit 1)
-    (in_bom yes) (on_board yes) (dnp no) (fields_autoplaced)
-    (property "Reference" "R1" (at 142.494 174.625 0)
-      (effects (font (size 1.27 1.27)) (justify left))
-    )
-    (property "Value" "91Ω" (at 142.494 177.165 0)
-      (effects (font (size 1.27 1.27)) (justify left))
-    )
-    (property "Footprint" "Capacitor_SMD:C_0805_2012Metric_Pad1.18x1.45mm_HandSolder" (at 138.684 175.895 90)
-      (effects (font (size 1.27 1.27)) hide)
-    )
-    (property "Datasheet" "~" (at 140.462 175.895 0)
+  (symbol (lib_id "Device:R") (at 140.462 175.133 0) (unit 1)
+    (in_bom yes) (on_board yes) (dnp no) (fields_autoplaced)
+    (property "Reference" "R1" (at 142.494 173.863 0)
+      (effects (font (size 1.27 1.27)) (justify left))
+    )
+    (property "Value" "91Ω" (at 142.494 176.403 0)
+      (effects (font (size 1.27 1.27)) (justify left))
+    )
+    (property "Footprint" "Capacitor_SMD:C_0805_2012Metric_Pad1.18x1.45mm_HandSolder" (at 138.684 175.133 90)
+      (effects (font (size 1.27 1.27)) hide)
+    )
+    (property "Datasheet" "~" (at 140.462 175.133 0)
       (effects (font (size 1.27 1.27)) hide)
     )
@@
       (effects (font (size 1.27 1.27)))
     )
-    (property "Footprint" "Capacitor_SMD:C_0402_1005Metric" (at 92.964 36.703 90)
-      (effects (font (size 1.27 1.27)) hide)
-    )
+    (property "Footprint" "Capacitor_SMD:C_0603_1608Metric" (at 92.964 36.703 90)
+      (effects (font (size 1.27 1.27)) hide)
+    )
