File: Matériel/PCB/Shémas.kicad_pcb (KiCad board)
At the start: 4 copper layers, 65 x 26 mm, 44 parts, among them J1 Conn_01x04_Socket, J3 Conn_01x04_Socket, J4 Conn_01x03_Socket, U1 MCP3221, U2 TCA9517, U3 XIAO ESP32C3, U5 LM117_TO3, U6 TJA1051T, U7 LM2674M-5.0

Commit message: Add files via upload
Parts:
- FB1: footprint Capacitor_SMD:C_0402_1005Metric -> Capacitor_SMD:C_0603_1608Metric
- moved FB1 0.71 mm to (102.3, 84.4), turned to 0 degrees
Connections:
- R6 pad 1: /RXD -> /TXD
- U3 pad 14: /TXD -> /RXD
Routing:
- net /RXD: track 5.18 -> 34.9 mm
- net /TXD: track 40.7 -> 11.5 mm
- net +3.3V: track 28.9 -> 30.6 mm
- net +5V: track 73.0 -> 71.4 mm
- net /SCLB: track 23.8 -> 25.1 mm
- net GND: track 85.9 -> 84.9 mm
- net /SCLA: track 11.7 -> 11.2 mm

Commit message: Pcb + code esp32 receive
gerber generate + recup du conne reception can
Parts:
- removed the G*** at (145.0, 82.7)
Changed lines of the file:
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@@
     )
-  )
-  (footprint "LOGO" (layer "B.Cu")
-    (at 145 82.7 180)
-    (attr board_only exclude_from_pos_files exclude_from_bom)
-    (fp_text reference "G***" (at 0 0) (layer "B.SilkS") hide
-        (effects (font (size 1.5 1.5) (thickness 0.3)) (justify mirror))
-    )
-    (fp_text value "LOGO" (at 0.75 0) (layer "B.SilkS") hide
-        (effects (font (size 1.5 1.5) (thickness 0.3)) (justify mirror))
-    )
-    (fp_poly
-      (pts
-        (xy 0.884389 2.944011)
-        (xy 0.895343 2.681028)
-        (xy 0.911549 2.500233)
-        (xy 0.938997 2.374334)
-        (xy 0.983676 2.276038)
-        (xy 1.051575 2.178053)
-        (xy 1.05283 2.176408)
-        (xy 1.269134 1.972484)
-        (xy 1.522891 1.857918)
-        (xy 1.792381 1.830597)
-        (xy 2.055886 1.88841)
-        (xy 2.291684 2.029245)
-        (xy 2.478058 2.250991)
-        (xy 2.51422 2.318485)
-        (xy 2.57648 2.478593)
-        (xy 2.612004 2.662268)
-        (xy 2.626446 2.904904)
-        (xy 2.627587 3.028059)
-        (xy 2.627587 3.503448)
-        (xy 2.846552 3.503448)
-        (xy 3.065518 3.503448)
-        (xy 3.065518 2.488552)
-        (xy 3.062808 2.08056)
-        (xy 3.052172 1.76476)
-        (xy 3.029847 1.523942)
-        (xy 2.992071 1.340893)
-        (xy 2.935082 1.198403)
-        (xy 2.855118 1.079261)
-        (xy 2.748416 0.966255)
-        (xy 2.728711 0.947686)
-        (xy 2.45777 0.764274)
-        (xy 2.126612 0.647063)
-        (xy 1.765021 0.599915)
-        (xy 1.402783 0.626691)
-        (xy 1.06968 0.731253)
-        (xy 1.067457 0.732299)
-        (xy 0.835465 0.858239)
-        (xy 0.660798 0.999156)
-        (xy 0.53596 1.171983)
-        (xy 0.453454 1.393656)
-        (xy 0.405783 1.681107)
-        (xy 0.385449 2.051273)
-        (xy 0.38319 2.277949)
-        (xy 0.38319 3.026655)
-        (xy -0.007989 2.99386)
-        (xy -0.445358 2.912293)
-        (xy -0.815071 2.750391)
-        (xy -1.11104 2.514348)
-        (xy -1.327177 2.210361)
-        (xy -1.457394 1.844627)
-        (xy -1.496064 1.4794)
-        (xy -1.470661 1.158814)
-        (xy -1.383458 0.910903)
-        (xy -1.224212 0.711757)
-        (xy -1.135941 0.638818)
-        (xy -0.972305 0.522385)
-        (xy -0.823188 0.436168)
-        (xy -0.666424 0.374414)
-        (xy -0.479846 0.331371)
-        (xy -0.241289 0.301286)
-        (xy 0.071414 0.278407)
-        (xy 0.301078 0.265887)
-        (xy 0.813362 0.234322)
-        (xy 1.231902 0.194262)
-        (xy 1.572363 0.141246)
-        (xy 1.850411 0.070816)
-        (xy 2.081709 -0.021488)
-        (xy 2.281924 -0.140127)
-        (xy 2.466718 -0.289559)
-        (xy 2.557523 -0.376511)
-        (xy 2.809578 -0.695039)
-        (xy 2.996083 -1.067625)
-        (xy 3.098333 -1.455552)
-        (xy 3.104923 -1.509492)
-        (xy 3.091691 -1.881708)
-        (xy 2.985351 -2.261474)
-        (xy 2.797508 -2.624375)
-        (xy 2.539769 -2.945998)
-        (xy 2.337799 -3.123206)
-        (xy 2.159249 -3.247276)
-        (xy 1.981413 -3.343843)
-        (xy 1.786804 -3.416625)
-        (xy 1.557931 -3.469341)
-        (xy 1.277306 -3.505709)
-        (xy 0.927438 -3.529447)
-        (xy 0.49084 -3.544275)
-        (xy 0.342134 -3.547505)
-        (xy -0.766379 -3.56943)
-        (xy -0.767279 -3.139564)
-        (xy -0.796663 -2.777843)
-        (xy -0.887808 -2.493835)
-        (xy -1.047754 -2.270428)
-        (xy -1.167268 -2.167431)
-        (xy -1.35694 -2.082216)
-        (xy -1.598266 -2.047689)
-        (xy -1.846797 -2.063934)
-        (xy -2.058082 -2.131033)
-        (xy -2.113831 -2.165667)
-        (xy -2.28469 -2.310481)
-        (xy -2.397393 -2.459479)
-        (xy -2.464744 -2.641875)
-        (xy -2.499542 -2.886881)
-        (xy -2.509864 -3.069439)
-        (xy -2.528996 -3.55819)
-        (xy -2.739284 -3.55819)
-        (xy -2.880581 -3.548487)
-        (xy -2.966789 -3.52444)
-        (xy -2.974601 -3.517134)
-        (xy -2.9822 -3.451633)
-        (xy -2.987965 -3.294904)
-        (xy -2.991596 -3.065191)
-        (xy -2.992791 -2.780739)
-        (xy -2.991517 -2.490733)
-        (xy -2.984873 -2.079352)
-        (xy -2.969175 -1.759935)
-        (xy -2.939329 -1.515034)
-        (xy -2.890244 -1.327201)
-        (xy -2.816829 -1.178988)
-        (xy -2.71399 -1.052947)
-        (xy -2.576638 -0.931632)
-        (xy -2.524666 -0.891038)
-        (xy -2.245979 -0.721932)
-        (xy -1.941448 -0.631569)
-        (xy -1.583382 -0.612938)
-        (xy -1.456462 -0.620691)
-        (xy -1.214383 -0.651627)
-        (xy -1.027103 -0.709033)
-        (xy -0.840256 -0.811036)
-        (xy -0.792677 -0.842012)
-        (xy -0.610972 -0.975666)
-        (xy -0.476502 -1.113668)
-        (xy -0.382471 -1.275071)
-        (xy -0.322083 -1.478926)
-        (xy -0.288542 -1.744286)
-        (xy -0.275055 -2.090202)
-        (xy -0.273706 -2.29699)
-        (xy -0.273706 -3.081396)
-        (xy 0.117472 -3.048601)
-        (xy 0.552019 -2.968448)
-        (xy 0.918177 -2.80794)
-        (xy 1.210898 -2.569541)
-        (xy 1.287343 -2.478372)
-        (xy 1.457273 -2.205344)
-        (xy 1.55593 -1.91093)
-        (xy 1.593603 -1.560992)
-        (xy 1.59469 -1.458799)
-        (xy 1.556915 -1.154379)
-        (xy 1.44002 -0.903424)
-        (xy 1.233827 -0.691025)
-        (xy 0.948925 -0.512912)
-        (xy 0.813168 -0.445484)
-        (xy 0.693052 -0.39719)
-        (xy 0.564785 -0.363723)
-        (xy 0.404576 -0.340774)
-        (xy 0.188632 -0.324037)
-        (xy -0.106839 -0.309204)
-        (xy -0.198405 -0.305181)
-        (xy -0.722055 -0.275935)
-        (xy -1.151614 -0.235406)
-        (xy -1.502237 -0.179456)
-        (xy -1.789084 -0.103946)
-        (xy -2.027312 -0.004735)
-        (xy -2.232079 0.122314)
-        (xy -2.418541 0.281341)
-        (xy -2.446327 0.308667)
-        (xy -2.725709 0.656427)
-        (xy -2.906959 1.032267)
-        (xy -2.993401 1.423116)
-        (xy -2.988356 1.815898)
-        (xy -2.895147 2.197542)
-        (xy -2.717095 2.554973)
-        (xy -2.457523 2.875118)
-        (xy -2.119754 3.144904)
-        (xy -1.707109 3.351258)
-        (xy -1.669612 3.365121)
-        (xy -1.548703 3.401151)
-        (xy -1.399678 3.429201)
-        (xy -1.2057 3.450766)
-        (xy -0.94993 3.467338)
-        (xy -0.615531 3.480412)
-        (xy -0.26518 3.4897)
-        (xy 0.865545 3.515671)
-      )
-      (stroke (width 0) (type solid)) (fill solid) (layer "B.SilkS"))
   )
   (footprint "Capacitor_SMD:C_0805_2012Metric_Pad1.18x1.45mm_HandSolder" (layer "B.Cu")
